File: Projeto_TCC.kicad_sch (KiCad schematic)
At the start: 58 parts, among them J1 Screw_Terminal_01x02, J2 Jack-DC, J3 Conn_01x15, J4 Conn_01x15, J5 Conn_01x04, J6 Conn_01x04, J7 Conn_01x04, J8 Conn_01x04, K1 AY1RC2, K2 AY1RC2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

Commit message: Battery tester TCC
Other:
- note added: "0-3V3"
- note added: "Voltage divider on sensor module"
Changed lines of the file:
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@@
   (junction (at 215.9 142.24) (diameter 0) (color 0 0 0 0)
   )
-  (junction (at 233.68 45.72) (diameter 0) (color 0 0 0 0)
-  )
   (junction (at 92.71 138.43) (diameter 0) (color 0 0 0 0)
   )
@@
     (stroke (width 0) (type default) (color 0 0 0 0))
   )
+  (polyline (pts (xy 109.22 125.73) (xy 173.99 125.73))
+    (stroke (width 0) (type default) (color 0 0 0 0))
+  )
+  (wire (pts (xy 66.04 95.25) (xy 77.47 95.25))
+    (stroke (width 0) (type default) (color 0 0 0 0))
+  )
+  (wire (pts (xy 187.96 152.4) (xy 187.96 148.59))
+    (stroke (width 0) (type default) (color 0 0 0 0))
+  )
+  (wire (pts (xy 125.73 71.12) (xy 125.73 73.66))
+    (stroke (width 0) (type default) (color 0 0 0 0))
+  )
+  (wire (pts (xy 96.52 138.43) (xy 92.71 138.43))
+    (stroke (width 0) (type default) (color 0 0 0 0))
+  )
+  (polyline (pts (xy 283.21 13.97) (xy 205.74 13.97))
+    (stroke (width 0) (type default) (color 0 0 0 0))
+  )
+  (wire (pts (xy 34.29 45.72) (xy 39.37 45.72))
+    (stroke (width 0) (type default) (color 0 0 0 0))
+  )
+  (polyline (pts (xy 173.99 193.04) (xy 109.22 193.04))
+    (stroke (width 0) (type default) (color 0 0 0 0))
+  )
+  (wire (pts (xy 96.52 166.37) (xy 96.52 167.64))
+    (stroke (width 0) (type default) (color 0 0 0 0))
+  )
+  (wire (pts (xy 215.9 140.97) (xy 218.44 140.97))
+    (stroke (width 0) (type default) (color 0 0 0 0))
+  )
+  (wire (pts (xy 267.97 95.25) (xy 267.97 101.6))
+    (stroke (width 0) (type default) (color 0 0 0 0))
+  )
+  (wire (pts (xy 181.61 58.42) (xy 181.61 60.96))
+    (stroke (width 0) (type default) (color 0 0 0 0))
+  )
+  (wire (pts (xy 267.97 91.44) (xy 267.97 95.25))
+    (stroke (width 0) (type default) (color 0 0 0 0))
+  )
+  (wire (pts (xy 85.09 78.74) (xy 85.09 71.12))
+    (stroke (width 0) (type default) (color 0 0 0 0))
+  )
+  (polyline (pts (xy 109.22 121.92) (xy 109.22 13.97))
+    (stroke (width 0) (type default) (color 0 0 0 0))
+  )
+  (wire (pts (xy 92.71 177.8) (xy 92.71 181.61))
+    (stroke (width 0) (type default) (color 0 0 0 0))
+  )
+  (wire (pts (xy 24.13 181.61) (xy 29.21 181.61))
+    (stroke (width 0) (type default) (color 0 0 0 0))
+  )
+  (wire (pts (xy 125.73 46.99) (xy 125.73 49.53))
+    (stroke (width 0) (type default) (color 0 0 0 0))
+  )
+  (wire (pts (xy 156.21 87.63) (xy 158.75 87.63))
+    (stroke (width 0) (type default) (color 0 0 0 0))
+  )
+  (wire (pts (xy 222.25 34.29) (xy 227.33 34.29))
+    (stroke (width 0) (type default) (color 0 0 0 0))
+  )
+  (wire (pts (xy 267.97 104.14) (xy 267.97 110.49))
+    (stroke (width 0) (type default) (color 0 0 0 0))
+  )
+  (wire (pts (xy 90.17 74.93) (xy 91.44 74.93))
+    (stroke (width 0) (type default) (color 0 0 0 0))
+  )
+  (wire (pts (xy 215.9 148.59) (xy 215.9 147.32))
+    (stroke (width 0) (type default) (color 0 0 0 0))
+  )
+  (wire (pts (xy 247.65 57.15) (xy 247.65 59.69))
+    (stroke (width 0) (type default) (color 0 0 0 0))
+  )
+  (polyline (pts (xy 110.49 13.97) (xy 200.66 13.97))
+    (stroke (width 0) (type default) (color 0 0 0 0))
+  )
   (wire (pts (xy 233.68 45.72) (xy 233.68 62.23))
-    (stroke (width 0) (type default) (color 0 0 0 0))
-  )
-  (polyline (pts (xy 109.22 125.73) (xy 173.99 125.73))
-    (stroke (width 0) (type default) (color 0 0 0 0))
-  )
-  (wire (pts (xy 66.04 95.25) (xy 77.47 95.25))
-    (stroke (width 0) (type default) (color 0 0 0 0))
-  )
-  (wire (pts (xy 187.96 152.4) (xy 187.96 148.59))
-    (stroke (width 0) (type default) (color 0 0 0 0))
-  )
-  (wire (pts (xy 125.73 71.12) (xy 125.73 73.66))
-    (stroke (width 0) (type default) (color 0 0 0 0))
-  )
-  (wire (pts (xy 96.52 138.43) (xy 92.71 138.43))
-    (stroke (width 0) (type default) (color 0 0 0 0))
-  )
-  (polyline (pts (xy 283.21 13.97) (xy 205.74 13.97))
-    (stroke (width 0) (type default) (color 0 0 0 0))
-  )
-  (wire (pts (xy 34.29 45.72) (xy 39.37 45.72))
-    (stroke (width 0) (type default) (color 0 0 0 0))
-  )
-  (polyline (pts (xy 173.99 193.04) (xy 109.22 193.04))
-    (stroke (width 0) (type default) (color 0 0 0 0))
-  )
-  (wire (pts (xy 96.52 166.37) (xy 96.52 167.64))
-    (stroke (width 0) (type default) (color 0 0 0 0))
-  )
-  (wire (pts (xy 215.9 140.97) (xy 218.44 140.97))
-    (stroke (width 0) (type default) (color 0 0 0 0))
-  )
-  (wire (pts (xy 267.97 95.25) (xy 267.97 101.6))
-    (stroke (width 0) (type default) (color 0 0 0 0))
-  )
-  (wire (pts (xy 181.61 58.42) (xy 181.61 60.96))
-    (stroke (width 0) (type default) (color 0 0 0 0))
-  )
-  (wire (pts (xy 267.97 91.44) (xy 267.97 95.25))
-    (stroke (width 0) (type default) (color 0 0 0 0))
-  )
-  (wire (pts (xy 85.09 78.74) (xy 85.09 71.12))
-    (stroke (width 0) (type default) (color 0 0 0 0))
-  )
-  (polyline (pts (xy 109.22 121.92) (xy 109.22 13.97))
-    (stroke (width 0) (type default) (color 0 0 0 0))
-  )
-  (wire (pts (xy 233.68 44.45) (xy 233.68 45.72))
-    (stroke (width 0) (type default) (color 0 0 0 0))
-  )
-  (wire (pts (xy 92.71 177.8) (xy 92.71 181.61))
-    (stroke (width 0) (type default) (color 0 0 0 0))
-  )
-  (wire (pts (xy 24.13 181.61) (xy 29.21 181.61))
-    (stroke (width 0) (type default) (color 0 0 0 0))
-  )
-  (wire (pts (xy 125.73 46.99) (xy 125.73 49.53))
-    (stroke (width 0) (type default) (color 0 0 0 0))
-  )
-  (wire (pts (xy 156.21 87.63) (xy 158.75 87.63))
-    (stroke (width 0) (type default) (color 0 0 0 0))
-  )
-  (wire (pts (xy 222.25 34.29) (xy 227.33 34.29))
-    (stroke (width 0) (type default) (color 0 0 0 0))
-  )
-  (wire (pts (xy 267.97 104.14) (xy 267.97 110.49))
-    (stroke (width 0) (type default) (color 0 0 0 0))
-  )
-  (wire (pts (xy 90.17 74.93) (xy 91.44 74.93))
-    (stroke (width 0) (type default) (color 0 0 0 0))
-  )
-  (wire (pts (xy 215.9 148.59) (xy 215.9 147.32))
-    (stroke (width 0) (type default) (color 0 0 0 0))
-  )
-  (wire (pts (xy 247.65 57.15) (xy 247.65 59.69))
-    (stroke (width 0) (type default) (color 0 0 0 0))
-  )
-  (polyline (pts (xy 110.49 13.97) (xy 200.66 13.97))
     (stroke (width 0) (type default) (color 0 0 0 0))
   )
@@
     (effects (font (size 2.5 2.5)) (justify left bottom))
   )
+  (text "Voltage divider on sensor module" (at 248.92 137.16 0)
+    (effects (font (size 1 1)) (justify left bottom))
+  )
   (text "Alimentação" (at 15.24 130.81 0)
     (effects (font (size 2.5 2.5)) (justify left bottom))
@@
     (effects (font (size 2.5 2.5)) (justify left bottom))
   )
+  (text "Voltage divider on sensor module" (at 198.12 137.16 0)
+    (effects (font (size 1 1)) (justify left bottom))
+  )
   (text "10W\n" (at 248.92 58.42 0)
     (effects (font (size 1 1)) (justify left bottom))
@@
     (effects (font (size 2.5 2.5)) (justify left bottom))
   )
+  (text "0-3V3" (at 179.07 144.78 0)
+    (effects (font (size 1 1)) (justify left bottom))
+  )
   (text "ADC2 CH4 on ESP32\n" (at 196.85 83.82 180)
     (effects (font (size 1 1)) (justify right bottom))
+  )
+  (text "0-3V3" (at 232.41 144.78 0)
+    (effects (font (size 1 1)) (justify left bottom))
   )
   (text "ADC2 CH0 on ESP32\n" (at 251.46 161.29 180)
@@
     (pin "1")
   )
-  (symbol (lib_id "power:GND") (at 256.54 62.23 0) (unit 1)
-    (in_bom yes) (on_board yes) (fields_autoplaced)
-    (property "Reference" "#PWR0104" (id 0) (at 256.54 68.58 0)
-      (effects (font (size 1.27 1.27)) hide)
-    )
-    (property "Value" "GND" (id 1) (at 256.54 67.31 0))
-    (property "Footprint" "" (id 2) (at 256.54 62.23 0)
-      (effects (font (size 1.27 1.27)) hide)
-    )
-    (property "Datasheet" "" (id 3) (at 256.54 62.23 0)
-      (effects (font (size 1.27 1.27)) hide)
-    )
-    (pin "1")
-  )
   (symbol (lib_id "Device:C") (at 172.72 99.06 0) (unit 1)
     (in_bom yes) (on_board yes) (fields_autoplaced)
@@
     (pin "9")
   )
+  (symbol (lib_id "power:GNDPWR") (at 256.54 62.23 0) (unit 1)
+    (in_bom yes) (on_board yes) (fields_autoplaced)
+    (property "Reference" "#PWR0104" (id 0) (at 256.54 67.31 0)
+      (effects (font (size 1.27 1.27)) hide)
+    )
+    (property "Value" "GNDPWR" (id 1) (at 256.413 67.31 0))
+    (property "Footprint" "" (id 2) (at 256.54 63.5 0)
+      (effects (font (size 1.27 1.27)) hide)
+    )
+    (property "Datasheet" "" (id 3) (at 256.54 63.5 0)
+      (effects (font (size 1.27 1.27)) hide)
+    )
+    (pin "1")
+  )
   (symbol (lib_id "power:GNDPWR") (at 234.95 111.76 0) (unit 1)
     (in_bom yes) (on_board yes) (fields_autoplaced)
@@
       (reference "#PWR0103") (unit 1) (value "GND") (footprint "")
     )
-    (path "/d2127ad6-de7f-4fd3-9225-e7ef9d59acec"
-      (reference "#PWR0104") (unit 1) (value "GND") (footprint "")
+    (path "/d6e2413e-9b6e-4768-9cec-30731c5b84f7"
+      (reference "#PWR0104") (unit 1) (value "GNDPWR") (footprint "")
     )
     (path "/3cb7a9da-6c9d-47d8-8036-58ae8e432832"
